File: DimLED.kicad_sch (KiCad schematic)
At the start: 14 parts, among them J1 Input Power Terminal, J2 DC005, J3 Conn_01x05, J4 Output LED Terminal, J5 Conn_01x03, SW1 IO BTN, SW2 RST BTN, U1 MP1584 Module, U2 ESP-01, U3 XY-MOS Module

Commit message: chore: general update
Parts:
- C1: Robu.in (none) -> https://robu.in/product/100nf-50v-through-hole-multilayer-c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
- C2: Robu.in (none) -> https://robu.in/product/hy1c102m080160cd288-hyncdz-1000uf-1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
- J1, J4: Robu.in (none) -> https://robu.in/product/xy306a-5-0-xinya-2-pin-screw-termin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
- J2: Robu.in (none) -> https://robu.in/product/dc-jack-005/
- R1, R2: Robu.in (none) -> https://robu.in/product/10k-ohm-0-25w-metal-film-resistor-p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
- SW1, SW2: Robu.in (none) -> https://robu.in/product/6x6x5-tactile-push-button-switch/
- U1: Robu.in (none) -> https://robu.in/product/mini-mp1584-dc-dc-3a-adjustable-buc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
- U2: Robu.in (none) -> https://robu.in/product/esp-01-esp8266-serial-wifi-wireless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
- U3: Robu.in (none) -> https://robu.in/product/switch-drive-high-power-mosfet-trig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
Changed lines of the file:
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@@
+			)
+		)
+		(property "Robu.in" "https://robu.in/product/switch-drive-high-power-mosfet-trigger-module/"
+			(at 210.82 55.88 0)
+			(effects
+				(font
+					(size 1.27 1.27)
+				)
+				(hide yes)
 			)
 		)
@@
 			)
 		)
+		(property "Robu.in" "https://robu.in/product/10k-ohm-0-25w-metal-film-resistor-pack-of-100/"
+			(at 132.08 124.46 0)
+			(effects
+				(font
+					(size 1.27 1.27)
+				)
+				(hide yes)
+			)
+		)
 		(pin "1"
 		)
@@
 		(property "Description" "Push button switch, generic, two pins"
 			(at 110.49 123.19 0)
+			(effects
+				(font
+					(size 1.27 1.27)
+				)
+				(hide yes)
+			)
+		)
+		(property "Robu.in" "https://robu.in/product/6x6x5-tactile-push-button-switch/"
+			(at 110.49 123.19 90)
 			(effects
 				(font
@@
 			)
 		)
+		(property "Robu.in" "https://robu.in/product/10k-ohm-0-25w-metal-film-resistor-pack-of-100/"
+			(at 110.49 132.08 0)
+			(effects
+				(font
+					(size 1.27 1.27)
+				)
+				(hide yes)
+			)
+		)
 		(pin "1"
 		)
@@
 		)
 		(property "Description" "Unpolarized capacitor"
+			(at 66.04 133.35 0)
+			(effects
+				(font
+					(size 1.27 1.27)
+				)
+				(hide yes)
+			)
+		)
+		(property "Robu.in" "https://robu.in/product/100nf-50v-through-hole-multilayer-ceramic-capacitor/"
 			(at 66.04 133.35 0)
 			(effects
@@
 			)
 		)
+		(property "Robu.in" "https://robu.in/product/xy306a-5-0-xinya-2-pin-screw-terminal-blockblue/"
+			(at 177.8 100.33 0)
+			(effects
+				(font
+					(size 1.27 1.27)
+				)
+				(hide yes)
+			)
+		)
 		(pin "2"
 		)
@@
 			)
 		)
+		(property "Robu.in" "https://robu.in/product/6x6x5-tactile-push-button-switch/"
+			(at 132.08 133.35 90)
+			(effects
+				(font
+					(size 1.27 1.27)
+				)
+				(hide yes)
+			)
+		)
 		(pin "2"
 		)
@@
 			)
 		)
+		(property "Robu.in" ""
+			(at 52.07 171.45 0)
+			(effects
+				(font
+					(size 1.27 1.27)
+				)
+				(hide yes)
+			)
+		)
 		(pin "2"
 		)
@@
 			)
 		)
+		(property "Robu.in" "https://robu.in/product/hy1c102m080160cd288-hyncdz-1000uf-16v-92m%cf%89100khz-%c2%b120-1-1a100khz-plugind8xl16mm-aluminum-electrolytic-capacitors-leaded-rohs/"
+			(at 81.28 133.35 0)
+			(effects
+				(font
+					(size 1.27 1.27)
+				)
+				(hide yes)
+			)
+		)
 		(pin "2"
 		)
@@
 			)
 		)
+		(property "Robu.in" "https://robu.in/product/mini-mp1584-dc-dc-3a-adjustable-buck-module-india/"
+			(at 128.27 48.26 0)
+			(effects
+				(font
+					(size 1.27 1.27)
+				)
+				(hide yes)
+			)
+		)
 		(pin "1"
 		)
@@
 			)
 		)
+		(property "Robu.in" ""
+			(at 180.34 39.37 0)
+			(effects
+				(font
+					(size 1.27 1.27)
+				)
+				(hide yes)
+			)
+		)
 		(pin "2"
 		)
@@
 		)
 		(property "Description" "Generic screw terminal, single row, 01x02, script generated (kicad-library-utils/schlib/autogen/connector/)"
+			(at 39.37 57.15 0)
+			(effects
+				(font
+					(size 1.27 1.27)
+				)
+				(hide yes)
+			)
+		)
+		(property "Robu.in" "https://robu.in/product/xy306a-5-0-xinya-2-pin-screw-terminal-blockblue/"
 			(at 39.37 57.15 0)
 			(effects
@@
 			)
 		)
+		(property "Robu.in" "https://robu.in/product/dc-jack-005/"
+			(at 48.26 40.64 0)
+			(effects
+				(font
+					(size 1.27 1.27)
+				)
+				(hide yes)
+			)
+		)
 		(pin "2"
 		)
@@
 			(at 77.47 100.33 0)
 			(effects
+				(font
+					(size 1.27 1.27)
+				)
+				(hide yes)
+			)
+		)
+		(property "Robu.in" "https://robu.in/product/esp-01-esp8266-serial-wifi-wireless-transceiver-module/"
+			(at 77.47 100.33 0)
+			(effects
